File: PCB/Eagle/OOK48_Interface.brd (EAGLE design)
At the start: 49.5 x 19 mm, 10 parts

Commit message: Add PCB data
Parts:
- removed E$10: (no value), diode:SOD123
- removed E$5: (no value), eagle-ltspice:R0805
- removed E$8: (no value), eagle-ltspice:C0805
- added C1: 100nF, eagle-ltspice:C0805
- added R3: 1K2, eagle-ltspice:R0805
- C2: value (none) -> 10uF
- J1: value (none) -> 16 SIL
- R1, R2: value (none) -> 47K
- renumbered E$1 to J1, E$2 to J2, E$3 to J3, E$4 to R1, E$6 to R2, E$7 to C2, E$9 to TR1
Connections:
- net S$4 renamed S$16
Routing:
- net S$16: track 114.2 -> 40.8 mm
- net S$4: track 0.00 -> 32.8 mm
- net S$15: track 51.2 -> 43.8 mm
- net S$9: track 2.50 -> 3.50 mm
- net S$13: track 14.2 -> 15.2 mm
Other:
- board size 49.5 x 19 mm -> 48 x 18.5 mm
- board text added: "0"
- board text added: "1"
- board text added: "19"
- board text added: "1PPS"
- board text added: "2"
- board text added: "20"
- board text added: "21"
- board text added: "26"
- board text added: "27"
- board text added: "28"
- board text added: "3"
- board text added: "3V3"
- board text added: "4"
- board text added: "5"
- board text added: "6"
- board text added: "7"
- board text added: "AF"
- board text added: "GND"
- board text added: "KEY"
- board text added: "Rx"
- board text added: "Tx"

Commit message: Add Tx Output
Parts:
- added TR2: (no value), linear:SOT23
- moved TR1 3.50 mm to (26.5, 9.25)
Routing:
- net S$11: track 2.00 -> 13.0 mm, vias 0 -> 1
- net S$17: track 0.00 -> 7.75 mm
- net S$7: track 11.2 -> 15.0 mm
- net S$19: track 0.00 -> 3.75 mm, vias 0 -> 1
- net S$4: track 32.8 -> 35.2 mm
- net S$6: track 5.25 -> 4.25 mm
- net S$5: track 6.00 -> 5.00 mm
- net S$16: track 40.8 -> 40.0 mm
Other:
- board text added: "TX"
Changed lines of the file:
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@@
 <wire x1="48" y1="18.5" x2="48" y2="0" width="0" layer="20"/>
 <wire x1="48" y1="0" x2="0" y2="0" width="0" layer="20"/>
-<text x="5.75" y="16.5" size="1" layer="25">AF</text>
-<text x="8.75" y="16.5" size="1" layer="25">GND</text>
-<text x="13" y="16.5" size="1" layer="25">KEY</text>
+<text x="4.75" y="16.5" size="1" layer="25">AF</text>
+<text x="7.25" y="16.5" size="1" layer="25">GND</text>
+<text x="10.75" y="16.5" size="1" layer="25">KEY</text>
 <text x="29.25" y="16.5" size="1" layer="25">3V3</text>
 <text x="32" y="16.5" size="1" layer="25">GND</text>
@@
 <text x="40" y="0.75" size="1" layer="25">1</text>
 <text x="42.5" y="0.75" size="1" layer="25">0</text>
+<text x="14" y="16.5" size="1" layer="25">TX</text>
 </plain>
 <attributes>
@@
 <attribute name="VALUE" x="17.52" y="10.79" size="1.27" layer="27" rot="R180"/>
 </element>
-<element name="TR1" library="linear" package="SOT23" value="" x="23" y="9.25" smashed="yes" rot="R90">
-<attribute name="NAME" x="24.155" y="12.345" size="1" layer="25" rot="R180"/>
-<attribute name="VALUE" x="26.175" y="7.345" size="1.27" layer="27" rot="R90"/>
+<element name="TR1" library="linear" package="SOT23" value="" x="26.5" y="9.25" smashed="yes" rot="R90">
+<attribute name="NAME" x="27.655" y="12.345" size="1" layer="25" rot="R180"/>
+<attribute name="VALUE" x="29.675" y="7.345" size="1.27" layer="27" rot="R90"/>
 </element>
 <element name="J2" library="bt_con-jst-xh" package="B4B-XH" value="" x="10.25" y="12.5" smashed="yes">
 <attribute name="NAME" x="2.5" y="12.56" size="1.27" layer="21" align="bottom-center"/>
 <attribute name="VALUE" x="10.25" y="8.69" size="1.27" layer="21" align="bottom-center"/>
+</element>
+<element name="TR2" library="linear" package="SOT23" value="" x="21" y="9.25" smashed="yes" rot="R90">
+<attribute name="NAME" x="22.155" y="12.345" size="1" layer="25" rot="R180"/>
+<attribute name="VALUE" x="24.175" y="7.345" size="1.27" layer="27" rot="R90"/>
 </element>
 </elements>
@@
 <wire x1="9" y1="14.75" x2="3" y2="14.75" width="1.016" layer="1"/>
 <wire x1="3" y1="10.75" x2="3" y2="14.75" width="1.016" layer="1"/>
-<wire x1="9" y1="14.75" x2="25.25" y2="14.75" width="1.016" layer="1"/>
-<wire x1="25.25" y1="14.75" x2="25.25" y2="10.5" width="1.016" layer="1"/>
+<wire x1="9" y1="14.75" x2="27.75" y2="14.75" width="1.016" layer="1"/>
+<wire x1="27.75" y1="14.75" x2="27.75" y2="10.5" width="1.016" layer="1"/>
 </signal>
 <signal name="S$5">
-<wire x1="25.25" y1="8.25" x2="24.25" y2="8.25" width="1.016" layer="1"/>
-<wire x1="25.25" y1="3.25" x2="25.25" y2="8.25" width="1.016" layer="1"/>
+<wire x1="27.75" y1="3.25" x2="27.75" y2="8.25" width="1.016" layer="1"/>
 </signal>
 <signal name="S$6">
-<wire x1="24.25" y1="10.25" x2="25.25" y2="10.25" width="1.016" layer="1"/>
-<wire x1="25.25" y1="10.25" x2="25.25" y2="14.5" width="1.016" layer="1"/>
+<wire x1="27.75" y1="10.25" x2="27.75" y2="14.5" width="1.016" layer="1"/>
 </signal>
 <signal name="S$7">
-<wire x1="14" y1="12.5" x2="20.25" y2="12.5" width="1.016" layer="1"/>
-<wire x1="20.25" y1="12.5" x2="20.25" y2="9.25" width="1.016" layer="1"/>
-<wire x1="20.25" y1="9.25" x2="22" y2="9.25" width="1.016" layer="1"/>
+<wire x1="14" y1="12.75" x2="14" y2="12.5" width="1.016" layer="1"/>
+<wire x1="14" y1="12.5" x2="16.5" y2="12.75" width="1.016" layer="1"/>
+<wire x1="16.5" y1="12.75" x2="25.25" y2="12.75" width="1.016" layer="1"/>
+<wire x1="25.25" y1="12.75" x2="25.25" y2="9.25" width="1.016" layer="1"/>
 </signal>
 <signal name="S$10">
@@
 <wire x1="4.75" y1="5.75" x2="5" y2="5.75" width="1.016" layer="1"/>
 </signal>
-<signal name="S$11">
-<contactref element="J2" pad="P$2"/>
-<wire x1="11.5" y1="12.5" x2="11.5" y2="14.5" width="1.016" layer="1"/>
-</signal>
 <signal name="S$16">
-<wire x1="7.5" y1="3.5" x2="7.5" y2="9.25" width="1.9304" layer="16"/>
-<wire x1="7.5" y1="9.25" x2="10" y2="9.25" width="1.9304" layer="16"/>
-<wire x1="10" y1="9.25" x2="10" y2="12.5" width="1.9304" layer="16"/>
-<wire x1="10" y1="12.5" x2="9" y2="12.5" width="1.9304" layer="16"/>
-<wire x1="10" y1="12.5" x2="11.5" y2="12.5" width="1.9304" layer="16"/>
+<wire x1="7.5" y1="3.5" x2="7.5" y2="7.5" width="1.9304" layer="16"/>
+<wire x1="7.5" y1="7.5" x2="9" y2="7.5" width="1.9304" layer="16"/>
+<wire x1="9" y1="7.5" x2="9" y2="12.5" width="1.9304" layer="16"/>
 <contactref element="J3" pad="P$4"/>
-<wire x1="33.5" y1="12.5" x2="33.5" y2="9.25" width="1.9304" layer="16"/>
-<wire x1="33.5" y1="9.25" x2="10" y2="9.25" width="1.9304" layer="16"/>
+<wire x1="33.5" y1="12.5" x2="33.5" y2="7.5" width="1.9304" layer="16"/>
+<wire x1="33.5" y1="7.5" x2="9" y2="7.5" width="1.9304" layer="16"/>
 </signal>
 <signal name="S$15">
@@
 <wire x1="3.25" y1="3.5" x2="4.75" y2="3.5" width="1.9304" layer="16"/>
 </signal>
+<signal name="S$17">
+<wire x1="25.25" y1="3.5" x2="25.25" y2="6.75" width="1.016" layer="1"/>
+<wire x1="25.25" y1="6.75" x2="22.25" y2="6.75" width="1.016" layer="1"/>
+<wire x1="22.25" y1="6.75" x2="22.25" y2="8.25" width="1.016" layer="1"/>
+</signal>
+<signal name="S$11">
+<contactref element="J2" pad="P$2"/>
+<wire x1="11.5" y1="12.5" x2="11.5" y2="10.5" width="1.016" layer="16"/>
+<wire x1="11.5" y1="10.5" x2="18.5" y2="10.5" width="1.016" layer="16"/>
+<wire x1="18.5" y1="10.5" x2="18.5" y2="11.25" width="1.016" layer="16"/>
+<wire x1="18.5" y1="11.25" x2="19.75" y2="11.25" width="1.016" layer="1"/>
+<wire x1="19.75" y1="11.25" x2="19.75" y2="9.25" width="1.016" layer="1"/>
+<via x="18.5" y="11.25" extent="1-16" drill="0.5"/>
+</signal>
+<signal name="S$19">
+<wire x1="22.25" y1="10.25" x2="23.75" y2="10.25" width="1.016" layer="1"/>
+<wire x1="23.75" y1="10.25" x2="23.75" y2="8" width="1.016" layer="16"/>
+<via x="23.75" y="10.25" extent="1-16" drill="0.5"/>
+</signal>
 </signals>
